File: cm4-bare-minimum/cm4-bare-minimum.kicad_sch (KiCad schematic)
At the start: 24 parts, among them J1 Micro_SD_Card_Det, J2 690-019-298-412, J3 THD-02-R, J4 USB4105-GF-A, J5 USB_OTG, U1 RT9742GGJ5, U2 RT9742SNGV, U3 FSUSB42MUX, U5 MagJack-A70-112-331N126

Commit message: Connector changed, Added Labels.
Changed HDMI connector to upright. Added labels for included components in schematic.
To Do: Create tracks in PCB Layout. Add jumper for wifi bluetooth signals.
Parts:
- removed J2: 690-019-298-412, CM4IO:EDAC 690-019-298-412, symbol CM4IO:HDMI_A_1.4
- added J6: G45A19170083HR, G45A19170083HR:AMPHENOL_G45A19170083HR, symbol G45A19170083HR:G45A19170083HR
Connections:
- net GND: now also J6.11, J6.17, J6.2, J6.5, J6.8, J6.SH1 (SHIELD), J6.SH2 (SHIELD__1), J6.SH3 (SHIELD__2), J6.SH4 (SHIELD__3)
- net HDMI0_CEC: now also J6.13
- net HDMI0_CK_N: now also J6.12
- net HDMI0_CK_P: now also J6.10
- net HDMI0_D0_N: now also J6.9
- net HDMI0_D0_P: now also J6.7
- net HDMI0_D1_N: now also J6.6
- net HDMI0_D1_P: now also J6.4
- net HDMI0_D2_N: now also J6.3
- net HDMI0_D2_P: now also J6.1
- net HDMI0_HOTPLUG: now also J6.19
- net HDMI0_SCL: now also J6.15
- net HDMI0_SDA: now also J6.16
- net HDMI_5v: now also J6.18
- no-connect marks 100 -> 99
Other:
- note added: "CM4"
- note added: "ETHERNET"
- note added: "HDMI"
- note added: "SD-CARD"
- note added: "USB"

Commit message: updated V1 bare minimum board
Initiated pcb layout for V1 board
Parts:
- removed C2, C4: 100n, Capacitor_SMD:C_0402_1005Metric, symbol Device:C
- removed J3: THD-02-R, Connector_PinHeader_2.54mm:PinHeader_2x02_P2.54mm_Vertical, symbol Connector_Generic:Conn_02x02_Odd_Even
- removed J6: G45A19170083HR, G45A19170083HR:AMPHENOL_G45A19170083HR, symbol G45A19170083HR:G45A19170083HR
- removed TP1: TestPoint, TestPoint:TestPoint_Pad_2.0x2.0mm, symbol Connector:TestPoint
- removed U2: RT9742SNGV, Package_TO_SOT_SMD:SOT-23, symbol CM4IO:RT9742SNGV
- added C1: 100n, Capacitor_SMD:C_0402_1005Metric, symbol Device:C
- added D2: LED Red, LED_SMD:LED_0603_1608Metric, symbol Device:LED
- added J1, J2: Conn_01x03, Connector_PinHeader_2.54mm:PinHeader_1x03_P2.54mm_Vertical, symbol Connector_Generic:Conn_01x03
- added J4: Molex 470531000, Connector:FanPinHeader_1x04_P2.54mm_Vertical, symbol Connector_Generic:Conn_01x04
- added J5: THD-20-R, Connector_PinHeader_2.54mm:PinHeader_2x20_P2.54mm_Vertical, symbol Connector_Generic:Conn_02x20_Odd_Even
- added J8: THD-02-R, Connector_PinHeader_2.54mm:PinHeader_2x02_P2.54mm_Vertical, symbol Connector_Generic:Conn_02x02_Odd_Even
- added R11: 1k, Resistor_SMD:R_0402_1005Metric, symbol Device:R
- added R13: 5.1k, Resistor_SMD:R_0402_1005Metric, symbol Device:R
- added R15, R16: 470R, Resistor_SMD:R_0402_1005Metric, symbol Device:R
- added R6, R7, R8: NC, Resistor_SMD:R_0402_1005Metric, symbol Device:R
- added R9: 36K 1%, Resistor_SMD:R_0402_1005Metric, symbol Device:R
- added U1: EMC2301-1-ACZL-TR, Package_SO:MSOP-8_3x3mm_P0.65mm, symbol CM4IO:EMC2301
- added U3: 74LVC1G07SE-7, Package_TO_SOT_SMD:SOT-353_SC-70-5, symbol CM4IO:74LVC1G07_copy
- R2: renamed from R1; value nf -> NC
- R3: renamed from R2; value nf -> NC
- R4, R5: value 470R -> NC; Field5 9239197 -> 9239278; Field6 RK73G1ETQTP4700D -> RK73G1ETQTP2201D; Field8 120887981 -> 120889581; Part Description Resistor 470R M1005 1% 63mW -> Resistor 2.2K M1005 1% 63mW
- renumbered C1 to C2, J1 to J3, J5 to J6, J4 to J7, R6 to R1, R3 to R10, R7 to R12, R8 to R14, U1 to U2, U3 to U4
Connections:
- net HDMI_5v is gone; now on an unnamed net: C3.1
- net BT_nDisable: now also R6.1
- net CM4_3V3: now also Module1.78 (GPIO_VREF(1.8v/3.3v_Input)), C1.1, D2.2 (A), J5.1 (Pin_1), J5.17 (Pin_17), R8.2, R9.2, U1.3 (VDD), U3.5 (VCC)
- net CM4_5V: now also J4.2 (Pin_2), J5.2 (Pin_2), J5.4 (Pin_4)
- net EEPROM_nWP: now also R5.1
- net GND: now also C1.2, J1.2 (Pin_2), J2.3 (Pin_3), J4.1 (Pin_1), J5.14 (Pin_14), J5.20 (Pin_20), J5.25 (Pin_25), J5.30 (Pin_30), J5.34 (Pin_34), J5.39 (Pin_39), J5.6 (Pin_6), J5.9 (Pin_9), R13.2, R6.2, R7.2, U1.4 (GND), U3.3 (GND); no longer Module1.15 (Ethernet_nLED3(3.3v)), Module1.17 (Ethernet_nLED2(3.3v))
- net Global_EN: now also J1.1 (Pin_1)
- net RUN_PG: now also J1.3 (Pin_3)
- net Reserved: now also R3.1
- net TR0_TAP: now also J8.3 (Pin_3)
- net TR1_TAP: now also J8.1 (Pin_1)
- net TR2_TAP: now also J8.2 (Pin_2)
- net TR3_TAP: now also J8.4 (Pin_4)
- net TRD0_P: no longer U5.1 (TRD0+)
- net WiFi_nDisable: now also R7.1
- net nPI_LED_PWR: now also U3.2
- net nRPIBOOT: now also J2.2 (Pin_2)
- net at U5.16 (LEDG_K): now also R15.1; no longer R4.1
- net at U5.18 (LEDY_K): now also R16.1; no longer R5.1
- net GPIO26: now reaches Module1.24 (GPIO26)
- net GPIO26: now also J5.37 (Pin_37)
- net GPIO21: now reaches Module1.25 (GPIO21)
- net GPIO21: now also J5.40 (Pin_40)
- net GPIO19: now reaches Module1.26 (GPIO19)
- net GPIO19: now also J5.35 (Pin_35)
- net GPIO20: now reaches Module1.27 (GPIO20)
- net GPIO20: now also J5.38 (Pin_38)
- net GPIO13: now reaches Module1.28 (GPIO13)
- net GPIO13: now also J5.33 (Pin_33)
- net GPIO16: now reaches Module1.29 (GPIO16)
- net GPIO16: now also J5.36 (Pin_36)
- net GPIO6: now reaches Module1.30 (GPIO6)
- net GPIO6: now also J5.31 (Pin_31)
- net GPIO12: now reaches Module1.31 (GPIO12)
- net GPIO12: now also J5.32 (Pin_32)
- net GPIO5: now reaches Module1.34 (GPIO5)
- net GPIO5: now also J5.29 (Pin_29)
- net ID_SC: now reaches Module1.35 (ID_SC)
- net ID_SC: now also J5.28 (Pin_28)
- net ID_SD: now reaches Module1.36 (ID_SD)
- net ID_SD: now also J5.27 (Pin_27)
- net GPIO7: now reaches Module1.37 (GPIO7)
- net GPIO7: now also J5.26 (Pin_26)
- net GPIO11: now reaches Module1.38 (GPIO11)
- net GPIO11: now also J5.23 (Pin_23)
- net GPIO8: now reaches Module1.39 (GPIO8)
- net GPIO8: now also J5.24 (Pin_24)
- net GPIO9: now reaches Module1.40 (GPIO9)
- net GPIO9: now also J5.21 (Pin_21)
- net GPIO25: now reaches Module1.41 (GPIO25)
- net GPIO25: now also J5.22 (Pin_22)
- net GPIO10: now reaches Module1.44 (GPIO10)
- net GPIO10: now also J5.19 (Pin_19)
- net GPIO24: now reaches Module1.45 (GPIO24)
- net GPIO24: now also J5.18 (Pin_18)
- net GPIO22: now reaches Module1.46 (GPIO22)
- net GPIO22: now also J5.15 (Pin_15)
- net GPIO23: now reaches Module1.47 (GPIO23)
- net GPIO23: now also J5.16 (Pin_16)
- net GPIO27: now reaches Module1.48 (GPIO27)
- net GPIO27: now also J5.13 (Pin_13)
- net GPIO18: now reaches Module1.49 (GPIO18)
- net GPIO18: now also J5.12 (Pin_12)
- net GPIO17: now reaches Module1.50 (GPIO17)
- net GPIO17: now also J5.11 (Pin_11)
- net GPIO15: now reaches Module1.51 (GPIO15)
- net GPIO15: now also J5.10 (Pin_10)
- net GPIO4: now reaches Module1.54 (GPIO4)
- net GPIO4: now also J5.7 (Pin_7)
- net GPIO14: now reaches Module1.55 (GPIO14)
- net GPIO14: now also J5.8 (Pin_8)
- net GPIO3: now reaches Module1.56 (GPIO3)
- net GPIO3: now also J5.5 (Pin_5)
- net GPIO2: now reaches Module1.58 (GPIO2)
- net GPIO2: now also J5.3 (Pin_3)
- net SD_VDD_Override: now reaches Module1.73 (SD_VDD_Override)
- net SD_VDD_Override: now also R4.1
- net SCL0: now reaches Module1.80 (SCL0)
- net SCL0: now also U1.2 (SCL)
- net SDA0: now reaches Module1.82 (SDA0)
- net SDA0: now also U1.1 (SDA)
- net AnalogIP1: now reaches Module1.94 (AnalogIP1)
- net AnalogIP1: now also J7.B5 (CC2), R13.1
- net AnalogIP0: now reaches Module1.96 (AnalogIP0)
- net AnalogIP0: now also J7.A5 (CC1), R14.1
- net HDMI0_CEC: no longer names the net of Module1.151 (HDMI0_CEC)
- net HDMI0_CK_N: no longer names the net of Module1.190 (HDMI0_CLK_N)
- net HDMI0_CK_P: no longer names the net of Module1.188 (HDMI0_CLK_P)
- net HDMI0_D0_N: no longer names the net of Module1.184 (HDMI0_TX0_N)
- net HDMI0_D0_P: no longer names the net of Module1.182 (HDMI0_TX0_P)
- net HDMI0_D1_N: no longer names the net of Module1.178 (HDMI0_TX1_N)
- net HDMI0_D1_P: no longer names the net of Module1.176 (HDMI0_TX1_P)
- net HDMI0_D2_N: no longer names the net of Module1.172 (HDMI0_TX2_N)
- net HDMI0_D2_P: no longer names the net of Module1.170 (HDMI0_TX2_P)
- net HDMI0_HOTPLUG: no longer names the net of Module1.153 (HDMI0_HOTPLUG)
- net HDMI0_SCL: no longer names the net of Module1.200 (HDMI0_SCL)
- net HDMI0_SDA: no longer names the net of Module1.199 (HDMI0_SDA)
- net VDAC_COMP: no longer names the net of Module1.111 (VDAC_COMP)
- net nEXTRST: no longer names the net of Module1.100 (nEXTRST)
- new net: J2.1 (Pin_1), R8.1
- new net: D2.1 (K), R11.1
- new net: R11.2, U3.4
- new net: J4.4 (Pin_4), U1.5 (PWM)
- new net: J4.3 (Pin_3), R9.1, U1.6 (TACH)
- new net ETH_LEDG: Module1.17 (Ethernet_nLED2(3.3v)), R15.2
- new net ETH_LEDY: Module1.15 (Ethernet_nLED3(3.3v)), R16.2
- no-connect marks 99 -> 82
Other:
- note added: "40Way GPIO Header"
- note added: "Also SMBUS alert IIC address : 0001_100x"
- note added: "FAN connector"
- note added: "FAN controler"
- note added: "IIC address : 0101_111x"
- note added: "MISCELLANEOUS"
- note added: "PWR LED"
- note added: "USB-OTG"
- note removed: "HDMI"
- note removed: "USB"
- company: (none) -> Rapid Analysis
- title: (none) -> V1 - CM4 Board
- moved on the sheet: C2, D1, J3, J6, J7, Module1A, Module1B, R1, R10, R12, R14, R2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
