File: Blade/Blade.kicad_sch (KiCad schematic)
At the start: 4 parts, among them J1 USB_C_Receptacle_USB2.0

Commit message: Fixing Blade Carrier Board
Parts:
- removed C2: 100n, Capacitor_SMD:C_0402_1005Metric, symbol Device:C
- removed J1: USB_C_Receptacle_USB2.0, Connector_USB:USB_C_Receptacle_GCT_USB4105-xx-A_16P_TopMnt_Horizontal, symbol Connector:USB_C_Receptacle_USB2.0_16P
- added J1: USB4105-GF-A, USB4105-GF-A:GCT_USB4105-GF-A, symbol USB4105-GF-A:USB4105-GF-A
- added R2: 5.1k, Resistor_SMD:R_0603_1608Metric_Pad0.98x0.95mm_HandSolder, symbol Device:R
- C1: value 100n -> 10u; footprint Capacitor_SMD:C_0402_1005Metric -> Capacitor_SMD:C_0805_2012Metric; Field4 Farnell -> Digikey; Field5 2611911 -> 490-14381-1-ND; Field6 RM EMK105 B7104KV-F -> GRM21BR71A106KA73L; Field7 TAIYO YUDEN EUROPE GMBH -> Murata; Field8 110091611 -> 111893011; Part Description 0.1uF 10% 16V Ceramic Capacitor X7R 0402 (1005 Metric) -> 10uF 10% 10V Ceramic Capacitor X7R 0805 (2012 Metric)
- R1: value 2.2K 1% -> 5.1k; footprint Resistor_SMD:R_0402_1005Metric -> Resistor_SMD:R_0603_1608Metric_Pad0.98x0.95mm_HandSolder; Digi-Key_PN (none) -> 311-5.10KHRCT-ND; Field4 Farnell -> (none); MPN (none) -> RC0603FR-075K1L; Manufacturer (none) -> Yageo; Part Description Resistor 2.2K M1005 1% 63mW -> (none)
Connections:
- net +5v: now also J1.A4_B9 (VBUS), J1.B4_A9 (VBUS__1); no longer R1.1
- net GND: now also J1.A1_B12 (GND), J1.B1_A12 (GND__1), J1.SH1 (SHELL_GND), J1.SH2 (SHELL_GND__1), J1.SH3 (SHELL_GND__2), J1.SH4 (SHELL_GND__3), R2.2
- new net: J1.B5 (CC2), R2.1
- new net: J1.A5 (CC1), R1.1
- no-connect marks 2 -> 6
Other:
- sheet CM5_GPIO ( Ethernet, GPIO, SDCARD) ports: added none; removed CC1, CC2
- sheet CM5_HighSpeed ports: added none; removed USB2_N, USB2_P
- note added: "Connectors ------- Ethernet SDCARD Jumpers Fan PWM GPIO"
- note added: "Connectors ------- USB-OTG CSI/DSI 0"
- note added: "USB-C (Power Only)"
- note removed: "Connectors ------- Ethernet SDCARD 40way RPI Jumpers Fan Battery"
- note removed: "Connectors ------- HDMI 0 HDMI 1 CSI/DSI 0 CSI/DSI 1"
- note removed: "Discharge Resistor Needed by some Type C PSUs"
- note removed: "TypeC Power connector"
