File: Blade/CM5_GPIO.kicad_sch (KiCad schematic)
At the start: 20 parts, among them J2 THD-02-R, J3 Micro_SD_Card_Det, J4 Conn_01x03, J5 JST_SHBM04B-SRSS-TB, J6 Conn_02x07_Odd_Even, SW1 Right angle Tact button, U1 TPD4EUSB30, U2 TPD4EUSB30, U3 MagJack-A70-112-331N126, U4 74LVC1G07SE-7, U5 RT9742GGJ5

Commit message: Fixing Blade Carrier Board
Parts:
- removed J6: Conn_02x07_Odd_Even, Connector_PinHeader_2.54mm:PinHeader_2x07_P2.54mm_Vertical, symbol Connector_Generic:Conn_02x07_Odd_Even
- removed SW1: Right angle Tact button, Button_Switch_THT:SW_Tactile_SPST_Angled_PTS645Vx58-2LFS, symbol Switch:SW_Push
- added J5: Conn_02x09_Odd_Even, Connector_PinHeader_2.54mm:PinHeader_2x09_P2.54mm_Vertical, symbol Connector_Generic:Conn_02x09_Odd_Even
- renumbered C3 to C2, C4 to C3, D2 to D1, D1 to D2, J5 to J3, J3 to J4, J4 to J6, R5 to R3, R2 to R4, R3 to R5, R4 to R6, U4 to U2, U2 to U3, U3 to U4
Connections:
- net EEPROM_nWP: now also J5.4 (Pin_4)
- net GND: now also J5.1 (Pin_1), J5.11 (Pin_11), J5.13 (Pin_13), J5.3 (Pin_3), J5.5 (Pin_5), J5.7 (Pin_7), J5.9 (Pin_9)
- net PMIC_ENABLE: now also J5.12 (Pin_12)
- net PWR_BUT: now also J5.14 (Pin_14)
- net SYNC_OUT: now also J5.6 (Pin_6)
- net USBOTG: now also J5.10 (Pin_10)
- net nRPIBOOT: now also J5.2 (Pin_2)
- net GPIO13: now reaches Module1.28 (GPIO13)
- net GPIO13: now also J5.16 (Pin_16)
- net GPIO12: now reaches Module1.31 (GPIO12)
- net GPIO12: now also J5.15 (Pin_15)
- net GPIO15: now reaches Module1.51 (GPIO15)
- net GPIO15: now also J5.18 (Pin_18)
- net GPIO14: now reaches Module1.55 (GPIO14)
- net GPIO14: now also J5.17 (Pin_17)
- net CC1: no longer names the net of Module1.94 (CC1)
- net CC2: no longer names the net of Module1.96 (CC2)
- no-connect marks 41 -> 39
Other:
- moved on the sheet: D1, D2, J3, J6, Module1A, R3, R4, U2
