File: Blade/PCIe-M2.kicad_sch (KiCad schematic)
At the start: 21 parts, among them J8 Bus_M.2_Socket_M, M1 M.2 Solder Nut, M2 M.2 Solder Nut, M3 M.2 Screw, U6 ASEK-32.768KHZ-L-R-T, U7 AP3441SHE-7B

Commit message: Fixing Blade Carrier Board
Parts:
- renumbered C11 to C10, C12 to C11, C13 to C12, C5 to C4, C6 to C5, C7 to C6, C8 to C7, C9 to C8, C10 to C9, J8 to J9, R7 to R10, R8 to R11, R9 to R12, R6 to R9, U6 to U7, U7 to U8
Changed lines of the file:
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@@
 		(on_board yes)
 		(dnp no)
-		(property "Reference" "#PWR031"
+		(property "Reference" "#PWR034"
 			(at 128.27 179.07 0)
 			(effects
@@
 			(project "Blade"
 				(path "/72f35eb9-d9c0-4fe9-94bf-2938cda04d14/2772383c-49e1-4a11-8cc0-86da9a747790"
-					(reference "#PWR031")
+					(reference "#PWR034")
 					(unit 1)
 				)
@@
 		(on_board yes)
 		(dnp no)
-		(property "Reference" "#PWR021"
+		(property "Reference" "#PWR024"
 			(at 189.23 137.16 0)
 			(effects
@@
 			(project "Blade"
 				(path "/72f35eb9-d9c0-4fe9-94bf-2938cda04d14/2772383c-49e1-4a11-8cc0-86da9a747790"
-					(reference "#PWR021")
+					(reference "#PWR024")
 					(unit 1)
 				)
@@
 		(on_board yes)
 		(dnp no)
-		(property "Reference" "C10"
+		(property "Reference" "C9"
 			(at 121.031 166.4716 0)
 			(effects
@@
 			(project "Blade"
 				(path "/72f35eb9-d9c0-4fe9-94bf-2938cda04d14/2772383c-49e1-4a11-8cc0-86da9a747790"
-					(reference "C10")
+					(reference "C9")
 					(unit 1)
 				)
@@
 		(on_board yes)
 		(dnp no)
-		(property "Reference" "C8"
+		(property "Reference" "C7"
 			(at 44.831 165.2016 0)
 			(effects
@@
 			(project "Blade"
 				(path "/72f35eb9-d9c0-4fe9-94bf-2938cda04d14/2772383c-49e1-4a11-8cc0-86da9a747790"
-					(reference "C8")
+					(reference "C7")
 					(unit 1)
 				)
@@
 		(on_board yes)
 		(dnp no)
-		(property "Reference" "#PWR034"
+		(property "Reference" "#PWR037"
 			(at 105.41 185.42 0)
 			(effects
@@
 			(project "Blade"
 				(path "/72f35eb9-d9c0-4fe9-94bf-2938cda04d14/2772383c-49e1-4a11-8cc0-86da9a747790"
-					(reference "#PWR034")
+					(reference "#PWR037")
 					(unit 1)
 				)
@@
 		(on_board yes)
 		(dnp no)
-		(property "Reference" "C5"
+		(property "Reference" "C4"
 			(at 222.631 133.4516 0)
 			(effects
@@
 			(project "Blade"
 				(path "/72f35eb9-d9c0-4fe9-94bf-2938cda04d14/2772383c-49e1-4a11-8cc0-86da9a747790"
-					(reference "C5")
+					(reference "C4")
 					(unit 1)
 				)
@@
 		(on_board yes)
 		(dnp no)
-		(property "Reference" "#PWR023"
+		(property "Reference" "#PWR026"
 			(at 60.96 175.26 0)
 			(effects
@@
 			(project "Blade"
 				(path "/72f35eb9-d9c0-4fe9-94bf-2938cda04d14/2772383c-49e1-4a11-8cc0-86da9a747790"
-					(reference "#PWR023")
+					(reference "#PWR026")
 					(unit 1)
 				)
@@
 		(on_board yes)
 		(dnp no)
-		(property "Reference" "C12"
+		(property "Reference" "C11"
 			(at 141.351 166.4716 0)
 			(effects
@@
 			(project "Blade"
 				(path "/72f35eb9-d9c0-4fe9-94bf-2938cda04d14/2772383c-49e1-4a11-8cc0-86da9a747790"
-					(reference "C12")
+					(reference "C11")
 					(unit 1)
 				)
@@
 		(on_board yes)
 		(dnp no)
-		(property "Reference" "J8"
+		(property "Reference" "J9"
 			(at 124.714 27.432 0)
 			(effects
@@
 			(project "Blade"
 				(path "/72f35eb9-d9c0-4fe9-94bf-2938cda04d14/2772383c-49e1-4a11-8cc0-86da9a747790"
-					(reference "J8")
+					(reference "J9")
 					(unit 1)
 				)
@@
 		(on_board yes)
 		(dnp no)
-		(property "Reference" "#PWR024"
+		(property "Reference" "#PWR027"
 			(at 24.13 177.8 0)
 			(effects
@@
 			(project "Blade"
 				(path "/72f35eb9-d9c0-4fe9-94bf-2938cda04d14/2772383c-49e1-4a11-8cc0-86da9a747790"
-					(reference "#PWR024")
+					(reference "#PWR027")
 					(unit 1)
 				)
@@
 		(on_board yes)
 		(dnp no)
-		(property "Reference" "C11"
+		(property "Reference" "C10"
 			(at 131.191 166.4716 0)
 			(effects
@@
 			(project "Blade"
 				(path "/72f35eb9-d9c0-4fe9-94bf-2938cda04d14/2772383c-49e1-4a11-8cc0-86da9a747790"
-					(reference "C11")
+					(reference "C10")
 					(unit 1)
 				)
@@
 		(on_board yes)
 		(dnp no)
-		(property "Reference" "R7"
+		(property "Reference" "R10"
 			(at 107.188 165.2016 0)
 			(effects
@@
 			(project "Blade"
 				(path "/72f35eb9-d9c0-4fe9-94bf-2938cda04d14/2772383c-49e1-4a11-8cc0-86da9a747790"
-					(reference "R7")
+					(reference "R10")
 					(unit 1)
 				)
@@
 		(on_board yes)
 		(dnp no)
-		(property "Reference" "R9"
+		(property "Reference" "R12"
 			(at 107.188 174.0916 0)
 			(effects
@@
 			(project "Blade"
 				(path "/72f35eb9-d9c0-4fe9-94bf-2938cda04d14/2772383c-49e1-4a11-8cc0-86da9a747790"
-					(reference "R9")
+					(reference "R12")
 					(unit 1)
 				)
@@
 		(on_board yes)
 		(dnp no)
-		(property "Reference" "R6"
+		(property "Reference" "R9"
 			(at 189.738 76.3016 0)
 			(effects
@@
 			(project "Blade"
 				(path "/72f35eb9-d9c0-4fe9-94bf-2938cda04d14/2772383c-49e1-4a11-8cc0-86da9a747790"
-					(reference "R6")
+					(reference "R9")
 					(unit 1)
 				)
@@
 		(dnp no)
 		(fields_autoplaced yes)
-		(property "Reference" "U7"
+		(property "Reference" "U8"
 			(at 59.69 151.13 0)
 			(effects
@@
 			(project "Blade"
 				(path "/72f35eb9-d9c0-4fe9-94bf-2938cda04d14/2772383c-49e1-4a11-8cc0-86da9a747790"
-					(reference "U7")
+					(reference "U8")
 					(unit 1)
 				)
@@
 		(on_board yes)
 		(dnp no)
-		(property "Reference" "#PWR026"
+		(property "Reference" "#PWR029"
 			(at 41.91 177.8 0)
 			(effects
@@
 			(project "Blade"
 				(path "/72f35eb9-d9c0-4fe9-94bf-2938cda04d14/2772383c-49e1-4a11-8cc0-86da9a747790"
-					(reference "#PWR026")
+					(reference "#PWR029")
 					(unit 1)
 				)
@@
 		(on_board yes)
 		(dnp no)
-		(property "Reference" "#PWR020"
+		(property "Reference" "#PWR023"
 			(at 127 130.81 0)
 			(effects
@@
 			(project "Blade"
 				(path "/72f35eb9-d9c0-4fe9-94bf-2938cda04d14/2772383c-49e1-4a11-8cc0-86da9a747790"
-					(reference "#PWR020")
+					(reference "#PWR023")
 					(unit 1)
 				)
@@
 		(on_board yes)
 		(dnp no)
-		(property "Reference" "#PWR032"
+		(property "Reference" "#PWR035"
 			(at 138.43 179.07 0)
 			(effects
@@
 			(project "Blade"
 				(path "/72f35eb9-d9c0-4fe9-94bf-2938cda04d14/2772383c-49e1-4a11-8cc0-86da9a747790"
-					(reference "#PWR032")
+					(reference "#PWR035")
 					(unit 1)
 				)
@@
 		(on_board yes)
 		(dnp no)
-		(property "Reference" "C13"
+		(property "Reference" "C12"
 			(at 151.511 166.4716 0)
 			(effects
@@
 			(project "Blade"
 				(path "/72f35eb9-d9c0-4fe9-94bf-2938cda04d14/2772383c-49e1-4a11-8cc0-86da9a747790"
-					(reference "C13")
+					(reference "C12")
 					(unit 1)
 				)
@@
 		(on_board yes)
 		(dnp no)
-		(property "Reference" "C9"
+		(property "Reference" "C8"
 			(at 98.171 165.2016 0)
 			(effects
@@
 			(project "Blade"
 				(path "/72f35eb9-d9c0-4fe9-94bf-2938cda04d14/2772383c-49e1-4a11-8cc0-86da9a747790"
-					(reference "C9")
+					(reference "C8")
 					(unit 1)
 				)
@@
 		(on_board yes)
 		(dnp no)
-		(property "Reference" "#PWR033"
+		(property "Reference" "#PWR036"
 			(at 148.59 179.07 0)
 			(effects
@@
 			(project "Blade"
 				(path "/72f35eb9-d9c0-4fe9-94bf-2938cda04d14/2772383c-49e1-4a11-8cc0-86da9a747790"
-					(reference "#PWR033")
+					(reference "#PWR036")
 					(unit 1)
 				)
@@
 		(on_board yes)
 		(dnp no)
-		(property "Reference" "#PWR030"
+		(property "Reference" "#PWR033"
 			(at 118.11 179.07 0)
 			(effects
@@
 			(project "Blade"
 				(path "/72f35eb9-d9c0-4fe9-94bf-2938cda04d14/2772383c-49e1-4a11-8cc0-86da9a747790"
-					(reference "#PWR030")
+					(reference "#PWR033")
 					(unit 1)
 				)
@@
 		(on_board yes)
 		(dnp no)
-		(property "Reference" "C6"
+		(property "Reference" "C5"
 			(at 27.051 165.2016 0)
 			(effects
@@
 			(project "Blade"
 				(path "/72f35eb9-d9c0-4fe9-94bf-2938cda04d14/2772383c-49e1-4a11-8cc0-86da9a747790"
-					(reference "C6")
+					(reference "C5")
 					(unit 1)
 				)
@@
 		(on_board yes)
 		(dnp no)
-		(property "Reference" "#PWR027"
+		(property "Reference" "#PWR030"
 			(at 50.8 177.8 0)
 			(effects
@@
 			(project "Blade"
 				(path "/72f35eb9-d9c0-4fe9-94bf-2938cda04d14/2772383c-49e1-4a11-8cc0-86da9a747790"
-					(reference "#PWR027")
+					(reference "#PWR030")
 					(unit 1)
 				)
@@
 		(on_board yes)
 		(dnp no)
-		(property "Reference" "#PWR029"
+		(property "Reference" "#PWR032"
 			(at 74.93 179.07 0)
 			(effects
@@
 			(project "Blade"
 				(path "/72f35eb9-d9c0-4fe9-94bf-2938cda04d14/2772383c-49e1-4a11-8cc0-86da9a747790"
-					(reference "#PWR029")
+					(reference "#PWR032")
 					(unit 1)
 				)
@@
 		(on_board yes)
 		(dnp no)
-		(property "Reference" "#PWR028"
+		(property "Reference" "#PWR031"
 			(at 69.85 179.07 0)
 			(effects
@@
 			(project "Blade"
 				(path "/72f35eb9-d9c0-4fe9-94bf-2938cda04d14/2772383c-49e1-4a11-8cc0-86da9a747790"
-					(reference "#PWR028")
+					(reference "#PWR031")
 					(unit 1)
 				)
@@
 		(on_board yes)
 		(dnp no)
-		(property "Reference" "R8"
+		(property "Reference" "R11"
 			(at 76.2 170.815 0)
 			(effects
@@
 			(project "Blade"
 				(path "/72f35eb9-d9c0-4fe9-94bf-2938cda04d14/2772383c-49e1-4a11-8cc0-86da9a747790"
-					(reference "R8")
+					(reference "R11")
 					(unit 1)
 				)
@@
 		(dnp no)
 		(fields_autoplaced yes)
-		(property "Reference" "U6"
+		(property "Reference" "U7"
 			(at 201.93 114.935 0)
 			(effects
@@
 			(project "Blade"
 				(path "/72f35eb9-d9c0-4fe9-94bf-2938cda04d14/2772383c-49e1-4a11-8cc0-86da9a747790"
-					(reference "U6")
+					(reference "U7")
 					(unit 1)
 				)
@@
 		(on_board yes)
 		(dnp no)
-		(property "Reference" "#PWR025"
+		(property "Reference" "#PWR028"
 			(at 33.02 177.8 0)
 			(effects
@@
 			(project "Blade"
 				(path "/72f35eb9-d9c0-4fe9-94bf-2938cda04d14/2772383c-49e1-4a11-8cc0-86da9a747790"
-					(reference "#PWR025")
+					(reference "#PWR028")
 					(unit 1)
 				)
@@
 		(on_board yes)
 		(dnp no)
-		(property "Reference" "C7"
+		(property "Reference" "C6"
 			(at 35.941 165.2016 0)
 			(effects
@@
 			(project "Blade"
 				(path "/72f35eb9-d9c0-4fe9-94bf-2938cda04d14/2772383c-49e1-4a11-8cc0-86da9a747790"
-					(reference "C7")
+					(reference "C6")
 					(unit 1)
 				)
@@
 		(on_board yes)
 		(dnp no)
-		(property "Reference" "#PWR022"
+		(property "Reference" "#PWR025"
 			(at 219.71 144.78 0)
 			(effects
@@
 			(project "Blade"
 				(path "/72f35eb9-d9c0-4fe9-94bf-2938cda04d14/2772383c-49e1-4a11-8cc0-86da9a747790"
-					(reference "#PWR022")
+					(reference "#PWR025")
 					(unit 1)
 				)
