File: Blade_v2/Blade_v2.kicad_pcb (KiCad board)
At the start: 2 copper layers, 120 x 40 mm, 44 parts, among them J1 USB_C_Receptacle_USB2.0, J2 THD-02-R, J3 Conn_02x08, J4 Micro_SD_Card_Det, J5 JST_SHBM04B-SRSS-TB, J6 Conn_01x22_Female, J7 Bus_M.2_Socket_M, U1 TPD4EUSB30, U2 TPD4EUSB30, U3 MagJack-A70-112-331N126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

Commit message: Update Blade_v2.kicad_pcb
Parts:
- moved R1 3.58 mm to (66.0, 47.1)
- moved R2 3.50 mm to (65.9, 44.0)
- moved R5 1.08 mm to (52.5, 61.0), turned to 0 degrees
- moved R4 0.95 mm to (55.4, 61.0), turned to 0 degrees
Routing:
- net /+3.3v: track 0.00 -> 186.2 mm, vias 0 -> 3
- net /+5v: track 66.7 -> 210.8 mm, vias 1 -> 5
- net /CM5_GPIO ( Ethernet, GPIO, SDCARD)/SCL0: track 0.00 -> 93.5 mm, vias 0 -> 2
- net /CM5_GPIO ( Ethernet, GPIO, SDCARD)/SDA0: track 0.00 -> 93.3 mm, vias 0 -> 2
- net /CM5_GPIO ( Ethernet, GPIO, SDCARD)/ETH_LEDY: track 0.00 -> 93.1 mm, vias 0 -> 2
- net /CM5_GPIO ( Ethernet, GPIO, SDCARD)/CAM_GPIO0: track 0.00 -> 92.4 mm, vias 0 -> 3
- net /CM5_GPIO ( Ethernet, GPIO, SDCARD)/SD_DAT2: track 0.00 -> 91.1 mm, vias 0 -> 4
- net /CM5_GPIO ( Ethernet, GPIO, SDCARD)/ETH_LEDG: track 0.00 -> 90.4 mm, vias 0 -> 2
- net /CM5_GPIO ( Ethernet, GPIO, SDCARD)/SD_DAT3: track 0.00 -> 88.1 mm, vias 0 -> 4
- net /CM5_GPIO ( Ethernet, GPIO, SDCARD)/SD_CMD: track 0.00 -> 87.1 mm, vias 0 -> 2
- net /CM5_GPIO ( Ethernet, GPIO, SDCARD)/SD_DAT1: track 0.00 -> 85.8 mm, vias 0 -> 2
- net /CM5_GPIO ( Ethernet, GPIO, SDCARD)/SD_CLK: track 0.00 -> 85.3 mm, vias 0 -> 2
- net /CM5_GPIO ( Ethernet, GPIO, SDCARD)/SD_DAT0: track 0.00 -> 84.9 mm, vias 0 -> 2
- net /CM5_GPIO ( Ethernet, GPIO, SDCARD)/nRPIBOOT: track 0.00 -> 78.1 mm, vias 0 -> 3
- net /CM5_GPIO ( Ethernet, GPIO, SDCARD)/nPWR_LED: track 0.00 -> 76.8 mm, vias 0 -> 4
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Other:
- outline, holes or cut-outs redrawn

Commit message: Blade_v2 Final revision
Parts:
- moved C1 1.78 mm to (65.7, 47.3)
- moved J1 1.78 mm to (54.4, 47.1)
- moved R1 1.78 mm to (66.1, 48.9)
- moved R2 1.78 mm to (66.1, 45.7)
- moved D1 1.00 mm to (93.2, 42.5)
- moved R3 1.00 mm to (91.2, 42.3)
- moved J5 0.86 mm to (107.8, 43.5)
Routing:
- net GND: track 91.4 -> 95.6 mm, vias 118 -> 125
- net Net-(Module1A-PI_nLED_Activity): track 74.5 -> 72.0 mm, vias 2 -> 4
- net /CM5_GPIO ( Ethernet, GPIO, SDCARD)/SDA0: track 93.3 -> 94.7 mm
- net /+5v: track 210.8 -> 211.7 mm
- net /+3.3v: track 186.2 -> 185.3 mm
- net /CM5_HighSpeed/USB2_P: track 98.3 -> 97.4 mm
- net /CM5_HighSpeed/USB2_N: track 98.3 -> 97.4 mm
- net /CM5_GPIO ( Ethernet, GPIO, SDCARD)/SCL0: track 93.5 -> 94.2 mm
- net Net-(J5-Pin_2): track 5.67 -> 4.97 mm
- net Net-(J5-Pin_4): track 13.9 -> 13.2 mm
Other:
- board text added: "PCB Edge"
- board text removed: "Analysis"
- board text removed: "Macquarie Park"
- board text removed: "Rapid"
