File: Blade_v2/Blade_v2.kicad_sch (KiCad schematic)
At the start: 4 parts, among them J1 USB_C_Receptacle_USB2.0

Commit message: Blade_v2 Final revision
Changed lines of the file:
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@@
+	)
+	(symbol
+		(lib_id "xerxes:LOGO")
+		(at 53.34 184.15 0)
+		(unit 1)
+		(exclude_from_sim no)
+		(in_bom yes)
+		(on_board yes)
+		(dnp no)
+		(fields_autoplaced yes)
+		(property "Reference" "#G1"
+			(at 53.34 181.8245 0)
+			(effects
+				(font
+					(size 1.27 1.27)
+				)
+				(hide yes)
+			)
+		)
+		(property "Value" "LOGO"
+			(at 53.34 186.4755 0)
+			(effects
+				(font
+					(size 1.27 1.27)
+				)
+				(hide yes)
+			)
+		)
+		(property "Footprint" ""
+			(at 53.34 184.15 0)
+			(effects
+				(font
+					(size 1.27 1.27)
+				)
+				(hide yes)
+			)
+		)
+		(property "Datasheet" ""
+			(at 53.34 184.15 0)
+			(effects
+				(font
+					(size 1.27 1.27)
+				)
+				(hide yes)
+			)
+		)
+		(property "Description" ""
+			(at 53.34 184.15 0)
+			(effects
+				(font
+					(size 1.27 1.27)
+				)
+				(hide yes)
+			)
+		)
+		(instances
+			(project ""
+				(path "/0855d192-8d15-45d1-ac78-b6f3f085784c"
+					(reference "#G1")
+					(unit 1)
+				)
+			)
+		)
 	)
 	(symbol
@@
 					(unit 1)
 				)
+			)
+		)
+	)
+	(symbol
+		(lib_id "RapidAnalysis_Logo:LOGO")
+		(at 53.34 161.29 0)
+		(unit 1)
+		(exclude_from_sim no)
+		(in_bom yes)
+		(on_board yes)
+		(dnp no)
+		(fields_autoplaced yes)
+		(property "Reference" "#G2"
+			(at 53.34 145.327 0)
+			(effects
+				(font
+					(size 1.27 1.27)
+				)
+				(hide yes)
+			)
+		)
+		(property "Value" "LOGO"
+			(at 53.34 177.253 0)
+			(effects
+				(font
+					(size 1.27 1.27)
+				)
+				(hide yes)
+			)
+		)
+		(property "Footprint" ""
+			(at 53.34 161.29 0)
+			(effects
+				(font
+					(size 1.27 1.27)
+				)
+				(hide yes)
+			)
+		)
+		(property "Datasheet" ""
+			(at 53.34 161.29 0)
+			(effects
+				(font
+					(size 1.27 1.27)
+				)
+				(hide yes)
+			)
+		)
+		(property "Description" ""
+			(at 53.34 161.29 0)
+			(effects
+				(font
+					(size 1.27 1.27)
+				)
+				(hide yes)
+			)
+		)
+		(instances
+			(project ""
+				(path "/0855d192-8d15-45d1-ac78-b6f3f085784c"
+					(reference "#G2")
+					(unit 1)
+				)

Commit message: Blade_V3 Commit
Other:
- note added: "Discharge Capacitor Needed by some Type C PSUs"
- note removed: "Discharge Resistor Needed by some Type C PSUs"
Changed lines of the file:
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@@
 		)
 	)
-	(text "Discharge Resistor\nNeeded by some\nType C PSUs"
+	(text "Discharge Capacitor\nNeeded by some\nType C PSUs"
 		(exclude_from_sim no)
 		(at 99.314 53.594 0)
