File: Blade_v3/Blade_v3.kicad_pcb (KiCad board)
At the start: 2 copper layers, 120 x 40 mm, 55 parts, among them J1 Conn_01x03, J2 Conn_01x03, J3 Conn_01x04, J4 Micro_SD_Card_Det, J5 THD-02-R, J6 Molex 470531000, J7 USB4105-GF-A, J8 USB_OTG, J9 Bus_M.2_Socket_M, U1 EMC2301-1-ACZL-TR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

Commit message: Latest Version Commit
Routing:
- net GND: track 73.5 -> 104.3 mm, vias 99 -> 113
- net /ETH_LEDY: track 83.9 -> 84.6 mm
- net /ETH_LEDG: track 86.4 -> 87.0 mm
